File: GemmaC3RC.kicad_sch (KiCad schematic)
At the start: 11 parts, among them J1 I2C_CH0, J2 I2C_CH1, J3 DC-Motor, J4 3.7V Battery, J5 Servo, J6 Pot, J7 Pot, J8 Ext1, J9 Ext2, U1 ESP32-C3_SUPERMINI

Commit message: Updated to ver 1.1
Bat is conneced to 3.3V and In1 io pin changed
Connections:
- net +3.3V: now also J4.1 (Pin_1), J5.2 (Pin_2), U2-Motor-Control1.4 (VCC)
- net GP21: now also U2-Motor-Control1.2 (IN3), U2-Motor-Control1.6 (IN1); no longer J8.1 (Pin_1)
- removed net +BATT: J4.1 (Pin_1), J5.2 (Pin_2), U1.5V, U2-Motor-Control1.4 (VCC)
- removed net MC_1: U1.6 (GPIO6), U2-Motor-Control1.2 (IN3), U2-Motor-Control1.6 (IN1)
- new net: J8.1 (Pin_1), U1.6 (GPIO6)
- no-connect marks 0 -> 1
Other:
- moved on the sheet: J8, J9
